File: PCB/divergence_meter/top_board.kicad_sch (KiCad schematic)
At the start: 11 parts

Commit message: working on PCB - itron board almost done
Connections:
- net at JS0.7 (Pin_7), itr1.10 (C), itr2.10 (C)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: no longer itr5.11 (DP), itr6.11 (DP), itr7.11 (DP), itr8.11 (DP)
- net at JS0.8 (Pin_8), itr1.11 (DP), itr2.11 (DP)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: now also itr5.11 (DP), itr6.11 (DP), itr7.11 (DP), itr8.11 (DP)
Changed lines of the file:
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@@
   (junction (at 134.62 60.96) (diameter 0) (color 0 0 0 0)
   )
-  (junction (at 87.63 72.39) (diameter 0) (color 0 0 0 0)
-  )
   (junction (at 93.98 57.15) (diameter 0) (color 0 0 0 0)
   )
@@
   (junction (at 134.62 128.27) (diameter 0) (color 0 0 0 0)
   )
+  (junction (at 88.9 72.39) (diameter 0) (color 0 0 0 0)
+  )
   (junction (at 121.92 132.08) (diameter 0) (color 0 0 0 0)
   )
@@
     (stroke (width 0) (type default) (color 0 0 0 0))
   )
+  (wire (pts (xy 76.2 72.39) (xy 88.9 72.39))
+    (stroke (width 0) (type default) (color 0 0 0 0))
+  )
   (wire (pts (xy 161.29 60.96) (xy 161.29 66.04))
     (stroke (width 0) (type default) (color 0 0 0 0))
@@
     (stroke (width 0) (type default) (color 0 0 0 0))
   )
-  (wire (pts (xy 87.63 93.98) (xy 87.63 72.39))
-    (stroke (width 0) (type default) (color 0 0 0 0))
-  )
   (wire (pts (xy 144.78 78.74) (xy 148.59 78.74))
     (stroke (width 0) (type default) (color 0 0 0 0))
@@
     (stroke (width 0) (type default) (color 0 0 0 0))
   )
-  (wire (pts (xy 76.2 72.39) (xy 87.63 72.39))
+  (wire (pts (xy 88.9 72.39) (xy 88.9 55.88))
     (stroke (width 0) (type default) (color 0 0 0 0))
   )
@@
     (stroke (width 0) (type default) (color 0 0 0 0))
   )
-  (wire (pts (xy 87.63 72.39) (xy 87.63 52.07))
+  (wire (pts (xy 87.63 52.07) (xy 87.63 93.98))
     (stroke (width 0) (type default) (color 0 0 0 0))
   )
@@
     (stroke (width 0) (type default) (color 0 0 0 0))
   )
-  (wire (pts (xy 88.9 78.74) (xy 88.9 55.88))
-    (stroke (width 0) (type default) (color 0 0 0 0))
-  )
+  (wire (pts (xy 88.9 78.74) (xy 88.9 72.39))
+    (stroke (width 0) (type default) (color 0 0 0 0))
+  )
