File: PCB/divergence_meter/divergence_meter.kicad_pcb (KiCad board)
At the start: 2 copper layers, 24 parts

Commit message: working on PCB - itron board almost done
Parts:
- added JPX1: Conn_02x04_Odd_Even, Connector_PinHeader_1.27mm:PinHeader_2x04_P1.27mm_Vertical, F.Cu at (129.5, 129.5)
- moved JG0 91.5 mm to (139.7, 66.0)
- moved JS0 10.6 mm to (50.2, 33.0)
- moved JP0 7.62 mm to (27.9, 53.3), turned to 180 degrees
- moved itr1 2.54 mm to (45.7, 50.8)
- moved itr2 2.54 mm to (73.7, 50.8)
- moved itr3 2.54 mm to (101.6, 50.8)
- moved itr4 2.54 mm to (129.5, 50.8)
- moved itr5 2.54 mm to (157.5, 50.8)
- moved itr6 2.54 mm to (185.4, 50.8)
- moved itr7 2.54 mm to (213.4, 50.8)
- moved itr8 2.54 mm to (241.3, 50.8)
Connections:
- JS0 pad 8: Net-(JS0-Pad8) -> Net-(itr5-Pad11)
- itr1 pad 11: Net-(JS0-Pad8) -> Net-(itr5-Pad11)
- itr2 pad 11: Net-(JS0-Pad8) -> Net-(itr5-Pad11)
- itr3 pad 11: Net-(JS0-Pad8) -> Net-(itr5-Pad11)
- itr4 pad 11: Net-(JS0-Pad8) -> Net-(itr5-Pad11)
- itr5 pad 11: Net-(JS0-Pad7) -> Net-(itr5-Pad11)
- itr6 pad 11: Net-(JS0-Pad7) -> Net-(itr5-Pad11)
- itr7 pad 11: Net-(JS0-Pad7) -> Net-(itr5-Pad11)
- itr8 pad 11: Net-(JS0-Pad7) -> Net-(itr5-Pad11)
Routing:
- net Net-(JS0-Pad7): track 0.00 -> 210.3 mm
- net Net-(JS0-Pad2): track 0.00 -> 210.3 mm
- net GND: track 0.00 -> 210.3 mm
- net Net-(JS0-Pad4): track 0.00 -> 205.4 mm
- net Net-(itr5-Pad11): track 0.00 -> 205.4 mm
- net Net-(JS0-Pad1): track 0.00 -> 205.4 mm
- net Net-(JG0-Pad1): track 0.00 -> 96.1 mm
- net Net-(JG0-Pad8): track 0.00 -> 94.8 mm
- net Net-(JG0-Pad2): track 0.00 -> 70.2 mm
- net Net-(JG0-Pad7): track 0.00 -> 68.6 mm
- net Net-(JG0-Pad3): track 0.00 -> 43.2 mm
- net Net-(JG0-Pad6): track 0.00 -> 42.5 mm
- net Net-(JG0-Pad4): track 0.00 -> 16.5 mm
- net Net-(JG0-Pad5): track 0.00 -> 15.2 mm

Commit message: itrons done, started logics
Parts:
- JG0, JP0, JS0: moved to B.Cu
- moved JRTC1 109.5 mm to (22.9, 167.0)
- moved JPX1 98.8 mm to (41.9, 175.3)
- moved JSW1 89.2 mm to (39.4, 121.3)
- moved JBT1 88.6 mm to (48.3, 129.5)
- moved JX2 83.9 mm to (36.8, 162.6)
- moved JR1 81.8 mm to (53.3, 188.0)
- moved UT2 75.6 mm to (105.4, 82.5), turned to -90 degrees
- moved JX1 65.3 mm to (43.2, 164.5)
- moved JG1 53.7 mm to (157.5, 176.5), turned to -90 degrees
- moved JS1 48.2 mm to (120.7, 99.1), turned to -90 degrees
- moved UT1 45.4 mm to (152.4, 165.1), turned to -90 degrees
- moved A1 41.0 mm to (108.0, 162.6)
- moved JP0 22.9 mm to (35.6, 31.8), turned to -90 degrees
- moved UR1 16.6 mm to (127.0, 170.2), turned to -90 degrees
- moved UR2 11.4 mm to (88.9, 128.3), turned to -90 degrees
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Connections:
- A1 pad 10: Net-(A1-Pad10) -> Net-(UR2-Pad11)
- A1 pad 5: Net-(A1-Pad5) -> Net-(UR1-Pad14)
- A1 pad 7: Net-(A1-Pad7) -> Net-(UR1-Pad11)
- UR1 pad 11: Net-(A1-Pad5) -> Net-(UR1-Pad11)
- UR1 pad 14: Net-(A1-Pad7) -> Net-(UR1-Pad14)
- UR2 pad 11: Net-(A1-Pad8) -> Net-(UR2-Pad11)
- UR2 pad 14: Net-(A1-Pad10) -> Net-(A1-Pad8)
Routing:
- net Net-(JS0-Pad8): track 205.4 -> 243.7 mm, vias 0 -> 1
- net Net-(JS0-Pad7): track 210.3 -> 244.6 mm
- net GND: track 210.3 -> 242.9 mm
- net Net-(JP0-Pad2): track 210.3 -> 237.4 mm
- net Net-(JS0-Pad1): track 205.4 -> 232.2 mm, vias 0 -> 1
- net Net-(JS0-Pad6): track 195.6 -> 217.8 mm
- net Net-(JS0-Pad2): track 210.3 -> 229.9 mm
- net Net-(JS0-Pad5): track 209.6 -> 226.2 mm
- net Net-(JS0-Pad4): track 205.4 -> 218.1 mm
- net Net-(JS0-Pad3): track 195.6 -> 206.5 mm
- net Net-(JG0-Pad6): track 42.5 -> 41.9 mm

Commit message: skoro hotova horní deska
Parts:
- moved itr8 64.8 mm to (176.5, 49.5)
- moved itr7 50.8 mm to (162.6, 49.5)
- moved itr6 36.9 mm to (148.6, 49.5)
- moved itr1 33.0 mm to (78.7, 49.5)
- moved JG0 30.3 mm to (123.2, 40.6)
- moved itr5 22.9 mm to (134.6, 49.5)
- moved itr2 19.3 mm to (92.9, 49.5)
- moved itr4 8.98 mm to (120.7, 49.5)
- moved itr3 5.24 mm to (106.7, 49.5)
Routing:
- net Net-(JS0-Pad7): track 244.6 -> 0.00 mm
- net Net-(JS0-Pad8): track 243.7 -> 0.00 mm, vias 1 -> 0
- net GND: track 242.9 -> 0.00 mm
- net Net-(JP0-Pad2): track 237.4 -> 0.00 mm
- net Net-(JS0-Pad1): track 232.2 -> 0.00 mm, vias 1 -> 0
- net Net-(JS0-Pad2): track 229.9 -> 0.00 mm
- net Net-(JS0-Pad5): track 226.2 -> 0.00 mm
- net Net-(JS0-Pad4): track 218.1 -> 0.00 mm
- net Net-(JS0-Pad6): track 217.8 -> 0.00 mm
- net Net-(JS0-Pad3): track 206.5 -> 0.00 mm
- net Net-(JG0-Pad1): track 96.1 -> 0.00 mm
- net Net-(JG0-Pad8): track 94.8 -> 0.00 mm
- net Net-(JG0-Pad2): track 70.2 -> 0.00 mm
- net Net-(JG0-Pad7): track 68.6 -> 0.00 mm
- net Net-(JG0-Pad3): track 43.2 -> 0.00 mm
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