File: PCB/LOGIC/divergence_meter.kicad_pcb (KiCad board)
At the start: 2 copper layers, 13 parts

Commit message: fakt nevim
Parts:
- UT1, UT2: moved to B.Cu
- moved JS1 60.4 mm to (97.8, 38.1), turned to -90 degrees
- moved UT2 59.3 mm to (87.6, 47.0), turned to 90 degrees
- moved JG1 43.2 mm to (165.1, 52.1), turned to -90 degrees
- moved UT1 25.8 mm to (154.9, 61.8), turned to 90 degrees
