File: PCB/TOP BOARD/divergence_meter.kicad_pcb (KiCad board)
At the start: 2 copper layers, 11 parts

Commit message: Dokončena horní deska
Parts:
- JG1, JP1, JS1: moved to B.Cu
- moved JG1 63.8 mm to (142.2, 120.7), turned to -90 degrees
- moved JP1 21.6 mm to (100.3, 116.8)
- turned JS1 to -90 degrees
Routing:
- net Net-(JG1-Pad1): track 0.00 -> 45.6 mm
- net Net-(JG1-Pad8): track 0.00 -> 42.9 mm
- net Net-(JG1-Pad2): track 0.00 -> 34.1 mm
- net Net-(JG1-Pad7): track 0.00 -> 32.8 mm
- net Net-(JG1-Pad3): track 0.00 -> 22.8 mm
- net Net-(JG1-Pad6): track 0.00 -> 21.4 mm
- net Net-(JP1-Pad1): track 140.6 -> 121.8 mm
- net Net-(JP1-Pad2): track 123.6 -> 111.8 mm
- net Net-(JG1-Pad4): track 0.00 -> 11.3 mm
- net Net-(JG1-Pad5): track 0.00 -> 10.7 mm
- net Net-(JS1-Pad7): track 157.4 -> 156.5 mm
Other:
- board outline added: 120.6 x 38.1 mm
- board text added: "@Toohka"
