File: PCB/TOP BOARD/divergence_meter.kicad_sch (KiCad schematic)
At the start: 11 parts

Commit message: Dokončena horní deska
Other:
- company: Projected by Toohka / Okarisu -> Made by Toohka / Okarisu
Changed lines of the file:
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@@
     (title "Divergence Meter - logic board")
     (date "2022")
-    (company "Projected by Toohka / Okarisu")
+    (company "Made by Toohka / Okarisu")
   )
   (junction (at 189.23 100.33) (diameter 0) (color 0 0 0 0)
