File: PCB/divergence_meter_logic/divergence_meter_logic.kicad_sch (KiCad schematic)
At the start: 16 parts

Commit message: remake pcb
Parts:
- removed JP3: 30V, symbol Connector_Generic:Conn_01x02
- added D1, D10, D11, D12, D13, D14, D15, D16, D2, D3, D4, D5, D6, D7, D8, D9: 1N4148, symbol Device:D
- added Q1, Q10, Q11, Q12, Q13, Q14, Q15, Q16, Q2, Q3, Q4, Q5, Q6, Q7, Q8, Q9: BC547, Package_TO_SOT_THT:TO-92_Inline, symbol Transistor_BJT:BC547
- added R1, R10, R11, R12, R13, R14, R15, R16, R2, R3, R4, R5, R6, R7, R8, R9: 100k, symbol Device:R
- JG1, JS1: footprint Connector_PinHeader_2.54mm:PinHeader_1x08_P2.54mm_Vertical -> Connector_PinSocket_2.54mm:PinSocket_1x08_P2.54mm_Vertical
- JRTC1: footprint Connector_PinHeader_2.54mm:PinHeader_1x06_P2.54mm_Vertical -> Connector_PinSocket_2.54mm:PinSocket_1x06_P2.54mm_Vertical
Connections:
- net +5V: no longer UR1.10 (~{SRCLR}), UR1.16 (VCC), UR2.10 (~{SRCLR}), UR2.16 (VCC)
- net GND: no longer JSW1.2 (Pin_2), JSW1.4 (Pin_4), JSW1.6 (Pin_6)
- net GND1: no longer UR1.13 (~{OE}), UR1.8 (GND), UR2.13 (~{OE}), UR2.8 (GND)
- net at UT1.10 (COM): no longer UT2.10 (COM)
- net at UT2.11 (O8): now also D10.1 (K), Q10.2 (B), R10.1; no longer JS1.8 (Pin_8)
- net at UT2.12 (O7): now also D12.1 (K), Q12.2 (B), R12.1; no longer JS1.7 (Pin_7)
- net at UT2.13 (O6): now also D14.1 (K), Q14.2 (B), R14.1; no longer JS1.6 (Pin_6)
- net at UT2.14 (O5): now also D16.1 (K), Q16.2 (B), R16.1; no longer JS1.5 (Pin_5)
- net at UT2.15 (O4): now also D15.1 (K), Q15.2 (B), R15.1; no longer JS1.4 (Pin_4)
- net at UT2.16 (O3): now also D13.1 (K), Q13.2 (B), R13.1; no longer JS1.3 (Pin_3)
- net at UT2.17 (O2): now also D11.1 (K), Q11.2 (B), R11.1; no longer JS1.2 (Pin_2)
- net at UT2.18 (O1): now also D9.1 (K), Q9.2 (B), R9.1; no longer JS1.1 (Pin_1)
- net at A1.10 (D7): no longer UR2.11 (SRCLK)
- net at A1.5 (D2): no longer UR1.14 (SER)
- net at A1.6 (D3): no longer UR1.12 (RCLK)
- net at A1.7 (D4): no longer UR1.11 (SRCLK)
- net at A1.8 (D5): no longer UR2.14 (SER)
- net at A1.9 (D6): no longer UR2.12 (RCLK)
- net at UT1.11 (O8): now also D2.1 (K), Q2.2 (B), R2.1; no longer JG1.8 (Pin_8)
- net at UT1.12 (O7): now also D4.1 (K), Q4.2 (B), R4.1; no longer JG1.7 (Pin_7)
- net at UT1.13 (O6): now also D6.1 (K), Q6.2 (B), R6.1; no longer JG1.6 (Pin_6)
- net at UT1.14 (O5): now also D8.1 (K), Q8.2 (B), R8.1; no longer JG1.5 (Pin_5)
- net at UT1.15 (O4): now also D7.1 (K), Q7.2 (B), R7.1; no longer JG1.4 (Pin_4)
- net at UT1.16 (O3): now also D5.1 (K), Q5.2 (B), R5.1; no longer JG1.3 (Pin_3)
- net at JG1.2 (Pin_2): now also JG1.1 (Pin_1), D1.2 (A), D3.2 (A), Q1.3 (E), Q3.3 (E); no longer UT1.17 (O2)
- net at UT1.18 (O1): now also D1.1 (K), Q1.2 (B), R1.1; no longer JG1.1 (Pin_1)
- new net: D4.2 (A), JG1.7 (Pin_7), Q4.3 (E)
- new net: D10.2 (A), JS1.8 (Pin_8), Q10.3 (E)
- new net: D12.2 (A), JS1.7 (Pin_7), Q12.3 (E)
- new net: D8.2 (A), JG1.5 (Pin_5), Q8.3 (E)
- new net: D11.2 (A), D9.2 (A), JS1.1 (Pin_1), JS1.2 (Pin_2), Q11.3 (E), Q9.3 (E)
- new net: D3.1 (K), Q3.2 (B), R3.1, UT1.17 (O2)
- new net: D6.2 (A), JG1.6 (Pin_6), Q6.3 (E)
- new net: D15.2 (A), JS1.4 (Pin_4), Q15.3 (E)
- new net: D2.2 (A), JG1.8 (Pin_8), Q2.3 (E)
- new net: D14.2 (A), JS1.6 (Pin_6), Q14.3 (E)
- new net: D7.2 (A), JG1.4 (Pin_4), Q7.3 (E)
- new net: D5.2 (A), JG1.3 (Pin_3), Q5.3 (E)
- new net: D13.2 (A), JS1.3 (Pin_3), Q13.3 (E)
- new net: D16.2 (A), JS1.5 (Pin_5), Q16.3 (E)
- new net: JSW1.2 (Pin_2), JSW1.4 (Pin_4), JSW1.6 (Pin_6)
- new net +28V: Q1.1 (C), Q10.1 (C), Q11.1 (C), Q12.1 (C), Q13.1 (C), Q14.1 (C), Q15.1 (C), Q16.1 (C), Q2.1 (C), Q3.1 (C), Q4.1 (C), Q5.1 (C), Q6.1 (C), Q7.1 (C), Q8.1 (C), Q9.1 (C), R1.2, R10.2, R11.2, R12.2, R13.2, R14.2, R15.2, R16.2, R2.2, R3.2, R4.2, R5.2, R6.2, R7.2, R8.2, R9.2
- no-connect marks 12 -> 13
Other:
- moved on the sheet: A1, JBT1, JG1, JP2, JPX1, JR1, JRTC1, JSW1, JX1, UR1, UT1

Commit message: code rework - display & time
Parts:
- D1, D10, D11, D12, D13, D14, D15, D16, D2, D3, D4, D5, D6, D7, D8, D9: footprint (none) -> Diode_THT:D_DO-34_SOD68_P5.08mm_Vertical_KathodeUp
Changed lines of the file:
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@@
     (property "Reference" "D4" (id 0) (at 195.58 53.34 0))
     (property "Value" "1N4148" (id 1) (at 195.58 48.26 0))
-    (property "Footprint" "" (id 2) (at 195.58 50.8 0)
+    (property "Footprint" "Diode_THT:D_DO-34_SOD68_P5.08mm_Vertical_KathodeUp" (id 2) (at 195.58 50.8 0)
       (effects (font (size 1.27 1.27)) hide)
     )
@@
     (property "Reference" "D12" (id 0) (at 195.58 115.57 0))
     (property "Value" "1N4148" (id 1) (at 195.58 110.49 0))
-    (property "Footprint" "" (id 2) (at 195.58 113.03 0)
+    (property "Footprint" "Diode_THT:D_DO-34_SOD68_P5.08mm_Vertical_KathodeUp" (id 2) (at 195.58 113.03 0)
       (effects (font (size 1.27 1.27)) hide)
     )
@@
     (property "Reference" "D8" (id 0) (at 228.6 53.34 0))
     (property "Value" "1N4148" (id 1) (at 228.6 48.26 0))
-    (property "Footprint" "" (id 2) (at 228.6 50.8 0)
+    (property "Footprint" "Diode_THT:D_DO-34_SOD68_P5.08mm_Vertical_KathodeUp" (id 2) (at 228.6 50.8 0)
       (effects (font (size 1.27 1.27)) hide)
     )
@@
     (property "Reference" "D3" (id 0) (at 195.58 30.48 0))
     (property "Value" "1N4148" (id 1) (at 195.58 35.56 0))
-    (property "Footprint" "" (id 2) (at 195.58 33.02 0)
+    (property "Footprint" "Diode_THT:D_DO-34_SOD68_P5.08mm_Vertical_KathodeUp" (id 2) (at 195.58 33.02 0)
       (effects (font (size 1.27 1.27)) hide)
     )
@@
     (property "Reference" "D10" (id 0) (at 179.07 115.57 0))
     (property "Value" "1N4148" (id 1) (at 179.07 110.49 0))
-    (property "Footprint" "" (id 2) (at 179.07 113.03 0)
+    (property "Footprint" "Diode_THT:D_DO-34_SOD68_P5.08mm_Vertical_KathodeUp" (id 2) (at 179.07 113.03 0)
       (effects (font (size 1.27 1.27)) hide)
     )
@@
     (property "Reference" "D14" (id 0) (at 212.09 115.57 0))
     (property "Value" "1N4148" (id 1) (at 212.09 110.49 0))
-    (property "Footprint" "" (id 2) (at 212.09 113.03 0)
+    (property "Footprint" "Diode_THT:D_DO-34_SOD68_P5.08mm_Vertical_KathodeUp" (id 2) (at 212.09 113.03 0)
       (effects (font (size 1.27 1.27)) hide)
     )
@@
     (property "Reference" "D9" (id 0) (at 179.07 92.71 0))
     (property "Value" "1N4148" (id 1) (at 179.07 97.79 0))
-    (property "Footprint" "" (id 2) (at 179.07 95.25 0)
+    (property "Footprint" "Diode_THT:D_DO-34_SOD68_P5.08mm_Vertical_KathodeUp" (id 2) (at 179.07 95.25 0)
       (effects (font (size 1.27 1.27)) hide)
     )
@@
     (property "Reference" "D11" (id 0) (at 195.58 92.71 0))
     (property "Value" "1N4148" (id 1) (at 195.58 97.79 0))
-    (property "Footprint" "" (id 2) (at 195.58 95.25 0)
+    (property "Footprint" "Diode_THT:D_DO-34_SOD68_P5.08mm_Vertical_KathodeUp" (id 2) (at 195.58 95.25 0)
       (effects (font (size 1.27 1.27)) hide)
     )
@@
     (property "Reference" "D15" (id 0) (at 228.6 92.71 0))
     (property "Value" "1N4148" (id 1) (at 228.6 97.79 0))
-    (property "Footprint" "" (id 2) (at 228.6 95.25 0)
+    (property "Footprint" "Diode_THT:D_DO-34_SOD68_P5.08mm_Vertical_KathodeUp" (id 2) (at 228.6 95.25 0)
       (effects (font (size 1.27 1.27)) hide)
     )
@@
     (property "Reference" "D1" (id 0) (at 179.07 30.48 0))
     (property "Value" "1N4148" (id 1) (at 179.07 35.56 0))
-    (property "Footprint" "" (id 2) (at 179.07 33.02 0)
+    (property "Footprint" "Diode_THT:D_DO-34_SOD68_P5.08mm_Vertical_KathodeUp" (id 2) (at 179.07 33.02 0)
       (effects (font (size 1.27 1.27)) hide)
     )
@@
     (property "Reference" "D13" (id 0) (at 212.09 92.71 0))
     (property "Value" "1N4148" (id 1) (at 212.09 97.79 0))
-    (property "Footprint" "" (id 2) (at 212.09 95.25 0)
+    (property "Footprint" "Diode_THT:D_DO-34_SOD68_P5.08mm_Vertical_KathodeUp" (id 2) (at 212.09 95.25 0)
       (effects (font (size 1.27 1.27)) hide)
     )
@@
     (property "Reference" "D7" (id 0) (at 228.6 30.48 0))
     (property "Value" "1N4148" (id 1) (at 228.6 35.56 0))
-    (property "Footprint" "" (id 2) (at 228.6 33.02 0)
+    (property "Footprint" "Diode_THT:D_DO-34_SOD68_P5.08mm_Vertical_KathodeUp" (id 2) (at 228.6 33.02 0)
       (effects (font (size 1.27 1.27)) hide)
     )
@@
     (property "Reference" "D5" (id 0) (at 212.09 30.48 0))
     (property "Value" "1N4148" (id 1) (at 212.09 35.56 0))
-    (property "Footprint" "" (id 2) (at 212.09 33.02 0)
+    (property "Footprint" "Diode_THT:D_DO-34_SOD68_P5.08mm_Vertical_KathodeUp" (id 2) (at 212.09 33.02 0)
       (effects (font (size 1.27 1.27)) hide)
     )
@@
     (property "Reference" "D6" (id 0) (at 212.09 53.34 0))
     (property "Value" "1N4148" (id 1) (at 212.09 48.26 0))
-    (property "Footprint" "" (id 2) (at 212.09 50.8 0)
+    (property "Footprint" "Diode_THT:D_DO-34_SOD68_P5.08mm_Vertical_KathodeUp" (id 2) (at 212.09 50.8 0)
       (effects (font (size 1.27 1.27)) hide)
     )
@@
     (property "Reference" "D16" (id 0) (at 228.6 115.57 0))
     (property "Value" "1N4148" (id 1) (at 228.6 110.49 0))
-    (property "Footprint" "" (id 2) (at 228.6 113.03 0)
+    (property "Footprint" "Diode_THT:D_DO-34_SOD68_P5.08mm_Vertical_KathodeUp" (id 2) (at 228.6 113.03 0)
       (effects (font (size 1.27 1.27)) hide)
     )
@@
     (property "Reference" "D2" (id 0) (at 179.07 53.34 0))
     (property "Value" "1N4148" (id 1) (at 179.07 48.26 0))
-    (property "Footprint" "" (id 2) (at 179.07 50.8 0)
+    (property "Footprint" "Diode_THT:D_DO-34_SOD68_P5.08mm_Vertical_KathodeUp" (id 2) (at 179.07 50.8 0)
       (effects (font (size 1.27 1.27)) hide)
     )
@@
     )
     (path "/9107f90e-86a8-40ce-9b18-211cf27a70d8"
-      (reference "D1") (unit 1) (value "1N4148") (footprint "")
+      (reference "D1") (unit 1) (value "1N4148") (footprint "Diode_THT:D_DO-34_SOD68_P5.08mm_Vertical_KathodeUp")
     )
     (path "/d5b0287f-b952-4991-86f0-1e143625e257"
-      (reference "D2") (unit 1) (value "1N4148") (footprint "")
+      (reference "D2") (unit 1) (value "1N4148") (footprint "Diode_THT:D_DO-34_SOD68_P5.08mm_Vertical_KathodeUp")
     )
     (path "/4473ae4b-17de-4783-9ee5-aa8b5fb26c31"
-      (reference "D3") (unit 1) (value "1N4148") (footprint "")
+      (reference "D3") (unit 1) (value "1N4148") (footprint "Diode_THT:D_DO-34_SOD68_P5.08mm_Vertical_KathodeUp")
     )
     (path "/03ee4e9c-a803-4d0a-9e4b-d1ae8ef82395"
-      (reference "D4") (unit 1) (value "1N4148") (footprint "")
+      (reference "D4") (unit 1) (value "1N4148") (footprint "Diode_THT:D_DO-34_SOD68_P5.08mm_Vertical_KathodeUp")
     )
     (path "/ace29780-620a-442d-8907-b6f176e74346"
-      (reference "D5") (unit 1) (value "1N4148") (footprint "")
+      (reference "D5") (unit 1) (value "1N4148") (footprint "Diode_THT:D_DO-34_SOD68_P5.08mm_Vertical_KathodeUp")
     )
     (path "/be19648a-6750-4954-8a32-c6391c900c04"
-      (reference "D6") (unit 1) (value "1N4148") (footprint "")
+      (reference "D6") (unit 1) (value "1N4148") (footprint "Diode_THT:D_DO-34_SOD68_P5.08mm_Vertical_KathodeUp")
     )
     (path "/a931beef-0434-43ea-b161-9da9846515fb"
-      (reference "D7") (unit 1) (value "1N4148") (footprint "")
+      (reference "D7") (unit 1) (value "1N4148") (footprint "Diode_THT:D_DO-34_SOD68_P5.08mm_Vertical_KathodeUp")
     )
     (path "/2b460761-7306-4378-8d53-ee61e57e3a1d"
-      (reference "D8") (unit 1) (value "1N4148") (footprint "")
+      (reference "D8") (unit 1) (value "1N4148") (footprint "Diode_THT:D_DO-34_SOD68_P5.08mm_Vertical_KathodeUp")
     )
     (path "/60d1331f-8661-4d5c-9efe-eaa62a189e36"
-      (reference "D9") (unit 1) (value "1N4148") (footprint "")
+      (reference "D9") (unit 1) (value "1N4148") (footprint "Diode_THT:D_DO-34_SOD68_P5.08mm_Vertical_KathodeUp")
     )
     (path "/49f48a05-a390-41f2-bbae-d57ade5cc480"
-      (reference "D10") (unit 1) (value "1N4148") (footprint "")
+      (reference "D10") (unit 1) (value "1N4148") (footprint "Diode_THT:D_DO-34_SOD68_P5.08mm_Vertical_KathodeUp")
     )
     (path "/7c55a9c7-f02a-448c-9b0f-3366ca54886e"
-      (reference "D11") (unit 1) (value "1N4148") (footprint "")
+      (reference "D11") (unit 1) (value "1N4148") (footprint "Diode_THT:D_DO-34_SOD68_P5.08mm_Vertical_KathodeUp")
     )
     (path "/29bc739c-fe98-491c-b302-1905388e913a"
-      (reference "D12") (unit 1) (value "1N4148") (footprint "")
+      (reference "D12") (unit 1) (value "1N4148") (footprint "Diode_THT:D_DO-34_SOD68_P5.08mm_Vertical_KathodeUp")
     )
     (path "/a8051ff8-49fd-44d0-91b7-28b3bb1e3ed9"
-      (reference "D13") (unit 1) (value "1N4148") (footprint "")
+      (reference "D13") (unit 1) (value "1N4148") (footprint "Diode_THT:D_DO-34_SOD68_P5.08mm_Vertical_KathodeUp")
     )
     (path "/5f45d6eb-b29e-4024-a373-ca132e673d9d"
-      (reference "D14") (unit 1) (value "1N4148") (footprint "")
+      (reference "D14") (unit 1) (value "1N4148") (footprint "Diode_THT:D_DO-34_SOD68_P5.08mm_Vertical_KathodeUp")
     )
     (path "/802fca80-1ef1-4cd6-8b2b-9c294f32ddf9"
-      (reference "D15") (unit 1) (value "1N4148") (footprint "")
+      (reference "D15") (unit 1) (value "1N4148") (footprint "Diode_THT:D_DO-34_SOD68_P5.08mm_Vertical_KathodeUp")
     )
     (path "/bf39fbfe-8b85-4d2a-b8fb-85a1a0a73b6a"
-      (reference "D16") (unit 1) (value "1N4148") (footprint "")
+      (reference "D16") (unit 1) (value "1N4148") (footprint "Diode_THT:D_DO-34_SOD68_P5.08mm_Vertical_KathodeUp")
     )
     (path "/6d5b0457-ef99-42c4-9903-52509f436e97"

Commit message: blah
Parts:
- removed JSW1: Conn_02x03_Odd_Even, Connector_PinHeader_2.54mm:PinHeader_2x03_P2.54mm_Vertical, symbol Connector_Generic:Conn_02x03_Odd_Even
- D1, D10, D11, D12, D13, D14, D15, D16, D2, D3, D4, D5, D6, D7, D8, D9: footprint Diode_THT:D_DO-34_SOD68_P5.08mm_Vertical_KathodeUp -> Diode_THT:D_DO-35_SOD27_P2.54mm_Vertical_KathodeUp
- R1, R10, R11, R12, R13, R14, R15, R16, R2, R3, R4, R5, R6, R7, R8, R9: footprint (none) -> Resistor_THT:R_Axial_DIN0204_L3.6mm_D1.6mm_P2.54mm_Vertical
Connections:
- net +28V: now also UT1.10 (COM), UT2.10 (COM)
- net +5V: now also UR1.10 (~{SRCLR}), UR1.16 (VCC), UR2.10 (~{SRCLR}), UR2.16 (VCC)
- net GND1: now also UR1.13 (~{OE}), UR1.8 (GND), UR2.13 (~{OE}), UR2.8 (GND)
- net at D1.2 (A), JG1.1 (Pin_1), Q1.3 (E): no longer D3.2 (A), JG1.2 (Pin_2), Q3.3 (E)
- net at D9.2 (A), JS1.1 (Pin_1), Q9.3 (E): no longer D11.2 (A), JS1.2 (Pin_2), Q11.3 (E)
- new net: D3.2 (A), JG1.2 (Pin_2), Q3.3 (E)
- new net: D11.2 (A), JS1.2 (Pin_2), Q11.3 (E)
- no-connect marks 13 -> 12
Other:
- moved on the sheet: D1, D10, D11, D12, D13, D14, D15, D16, D2, D3, D4, D5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

Commit message: wuzah
Parts:
- added SW1, SW2, SW3: SW_Push, symbol Switch:SW_Push
Connections:
- net at D9.1 (K), Q9.2 (B), R9.1: now also UT2.11 (O8); no longer UT2.18 (O1)
- net at D13.1 (K), Q13.2 (B), R13.1: now also UT2.13 (O6); no longer UT2.16 (O3)
- net at D10.1 (K), Q10.2 (B), R10.1: now also UT2.18 (O1); no longer UT2.11 (O8)
- net at D12.1 (K), Q12.2 (B), R12.1: now also UT2.17 (O2); no longer UT2.12 (O7)
- net at UR1.1 (QB): now also UT1.7 (I7); no longer UT1.2 (I2)
- net at UR1.15 (QA): now also UT1.8 (I8); no longer UT1.1 (I1)
- net at UR1.2 (QC): now also UT1.6 (I6); no longer UT1.3 (I3)
- net at UR1.3 (QD): now also UT1.5 (I5); no longer UT1.4 (I4)
- net at UR1.4 (QE): now also UT1.4 (I4); no longer UT1.5 (I5)
- net at UR1.5 (QF): now also UT1.3 (I3); no longer UT1.6 (I6)
- net at UR1.6 (QG): now also UT1.2 (I2); no longer UT1.7 (I7)
- net at UR1.7 (QH): now also UT1.1 (I1); no longer UT1.8 (I8)
- net at D11.1 (K), Q11.2 (B), R11.1: now also UT2.12 (O7); no longer UT2.17 (O2)
- net at D15.1 (K), Q15.2 (B), R15.1: now also UT2.14 (O5); no longer UT2.15 (O4)
- net at D14.1 (K), Q14.2 (B), R14.1: now also UT2.16 (O3); no longer UT2.13 (O6)
- net at D16.1 (K), Q16.2 (B), R16.1: now also UT2.15 (O4); no longer UT2.14 (O5)
Other:
- moved on the sheet: D10, D11, D12, D13, D14, D15, D16, D9, Q10, Q11, Q12, Q13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

Commit message: pcb rework
Parts:
- removed JBT1: Conn_01x06, Connector_PinHeader_2.54mm:PinHeader_1x06_P2.54mm_Vertical, symbol Connector_Generic:Conn_01x06
- removed JPX1: Conn_02x04_Odd_Even, Connector_PinHeader_2.54mm:PinHeader_2x04_P2.54mm_Vertical, symbol Connector_Generic:Conn_02x04_Odd_Even
- removed JR1: Conn_01x02, Connector_PinHeader_2.54mm:PinHeader_1x02_P2.54mm_Vertical, symbol Connector_Generic:Conn_01x02
- removed JX1: Conn_01x07, Connector_PinHeader_2.54mm:PinHeader_1x07_P2.54mm_Vertical, symbol Connector_Generic:Conn_01x07
- added H1, H2, H3, H4: MountingHole_Pad, MountingHole:MountingHole_3.5mm_Pad_Via, symbol Mechanical:MountingHole_Pad
- added J1: Conn_Coaxial_Power, symbol Connector:Conn_Coaxial_Power
- added JGND1: Conn_01x03, Connector_PinHeader_2.54mm:PinHeader_1x03_P2.54mm_Vertical, symbol Connector_Generic:Conn_01x03
- added SWR1: SW_Push, symbol Switch:SW_Push
- renumbered D12 to D10, D14 to D11, D16 to D12, D15 to D13, D13 to D14, D11 to D15, D9 to D16, D3 to D2, D5 to D3, D7 to D4, D8 to D5, D4 to D7, D2 to D8, D10 to D9, Q12 to Q10, Q14 to Q11, Q16 to Q12, Q15 to Q13, Q13 to Q14, Q11 to Q15, Q9 to Q16, Q3 to Q2, Q5 to Q3, Q7 to Q4, Q8 to Q5, Q4 to Q7, Q2 to Q8, Q10 to Q9, R12 to R10, R14 to R11, R16 to R12, R15 to R13, R13 to R14, R11 to R15, R9 to R16, R3 to R2, R5 to R3, R7 to R4, R8 to R5, R4 to R7, R2 to R8, R10 to R9
Connections:
- net GND: now also A1.29 (GND), JRTC1.1 (Pin_1), UR1.13 (~{OE}), UR1.8 (GND), UR2.13 (~{OE}), UR2.8 (GND), JGND1.3 (Pin_3), SWR1.2; no longer UT1.9 (GND), UT2.9 (GND)
- net GND1: no longer A1.29 (GND), A1.4 (GND), JRTC1.1 (Pin_1), UR1.13 (~{OE}), UR1.8 (GND), UR2.13 (~{OE}), UR2.8 (GND)
- net at A1.10 (D7): now also UR1.11 (SRCLK)
- net at A1.28 (~{RESET}): now also SWR1.1
- net at A1.5 (D2): now also UR2.14 (SER)
- net at A1.6 (D3): now also UR2.12 (RCLK)
- net at A1.7 (D4): now also UR2.11 (SRCLK)
- net at A1.8 (D5): now also UR1.14 (SER)
- net at A1.9 (D6): now also UR1.12 (RCLK)
- net at D9.2 (A), Q9.3 (E): now also JS1.1 (Pin_1); no longer JS1.8 (Pin_8)
- net at D10.2 (A), Q10.3 (E): now also JS1.2 (Pin_2); no longer JS1.7 (Pin_7)
- net at D16.2 (A), Q16.3 (E): now also JS1.8 (Pin_8); no longer JS1.1 (Pin_1)
- net at D13.2 (A), Q13.3 (E): now also JS1.5 (Pin_5); no longer JS1.4 (Pin_4)
- net at D11.2 (A), Q11.3 (E): now also JS1.3 (Pin_3); no longer JS1.6 (Pin_6)
- net at D15.2 (A), Q15.3 (E): now also JS1.7 (Pin_7); no longer JS1.2 (Pin_2)
- net at D14.2 (A), Q14.3 (E): now also JS1.6 (Pin_6); no longer JS1.3 (Pin_3)
- net at D12.2 (A), Q12.3 (E): now also JS1.4 (Pin_4); no longer JS1.5 (Pin_5)
- net at UR2.15 (QA): now also UT2.8 (I8); no longer UT2.1 (I1)
- net at UR2.1 (QB): now also UT2.7 (I7); no longer UT2.2 (I2)
- net at UR2.2 (QC): now also UT2.6 (I6); no longer UT2.3 (I3)
- net at UR2.3 (QD): now also UT2.5 (I5); no longer UT2.4 (I4)
- net at UR2.4 (QE): now also UT2.4 (I4); no longer UT2.5 (I5)
- net at UR2.5 (QF): now also UT2.3 (I3); no longer UT2.6 (I6)
- net at UR2.6 (QG): now also UT2.2 (I2); no longer UT2.7 (I7)
- net at UR2.7 (QH): now also UT2.1 (I1); no longer UT2.8 (I8)
- new net: H1.1, H2.1, H3.1, H4.1, JGND1.2 (Pin_2)
- new net +12V: J1.1 (In)
- new net GNDPWR: J1.2 (Ext), JGND1.1 (Pin_1)
- no-connect marks 12 -> 8
Other:
- company: Projected by Toohka / Okarisu -> Author: Okarisu (Toohka)
- moved on the sheet: A1, JP1, JP2, JRTC1, SW1, SW2, SW3

Commit message: pcb finishing
Parts:
- removed JGND1: Conn_01x03, Connector_PinHeader_2.54mm:PinHeader_1x03_P2.54mm_Vertical, symbol Connector_Generic:Conn_01x03
- removed JP1: 1V, symbol Connector_Generic:Conn_01x02
- removed JP2: 5V, symbol Connector_Generic:Conn_01x02
- added JP1: SolderJumper_3_Open, Jumper:SolderJumper-3_P1.3mm_Open_RoundedPad1.0x1.5mm_NumberLabels, symbol Jumper:SolderJumper_3_Open
- JRTC1: footprint Connector_PinSocket_2.54mm:PinSocket_1x06_P2.54mm_Vertical -> Connector_PinSocket_2.54mm:PinSocket_1x06_P2.54mm_Horizontal
- renumbered D8 to D1, D15 to D10, D14 to D11, D13 to D12, D12 to D13, D11 to D14, D10 to D15, D9 to D16, D7 to D2, D6 to D3, D5 to D4, D4 to D5, D3 to D6, D2 to D7, D1 to D8, D16 to D9, Q8 to Q1, Q15 to Q10, Q14 to Q11, Q13 to Q12, Q12 to Q13, Q11 to Q14, Q10 to Q15, Q9 to Q16, Q7 to Q2, Q6 to Q3, Q5 to Q4, Q4 to Q5, Q3 to Q6, Q2 to Q7, Q1 to Q8, Q16 to Q9, R8 to R1, R15 to R10, R14 to R11, R13 to R12, R12 to R13, R11 to R14, R10 to R15, R9 to R16, R7 to R2, R6 to R3, R5 to R4, R4 to R5, R3 to R6, R2 to R7, R1 to R8, R16 to R9
Connections:
- net GND: now also A1.4 (GND), JP1.3 (B)
- net GNDPWR: now also JP1.1 (A)
- net at D2.2 (A), Q2.3 (E): now also JG1.2 (Pin_2); no longer JG1.7 (Pin_7)
- net at H1.1, H2.1, H3.1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: now also JP1.2 (C)
- net at D8.2 (A), Q8.3 (E): now also JG1.8 (Pin_8); no longer JG1.1 (Pin_1)
- net at D16.2 (A), Q16.3 (E): now also JS1.8 (Pin_8); no longer JS1.1 (Pin_1)
- net at D15.2 (A), Q15.3 (E): now also JS1.7 (Pin_7); no longer JS1.2 (Pin_2)
- net at D4.2 (A), Q4.3 (E): now also JG1.4 (Pin_4); no longer JG1.5 (Pin_5)
- net at D9.2 (A), Q9.3 (E): now also JS1.1 (Pin_1); no longer JS1.8 (Pin_8)
- net at D7.2 (A), Q7.3 (E): now also JG1.7 (Pin_7); no longer JG1.2 (Pin_2)
- net at D3.2 (A), Q3.3 (E): now also JG1.3 (Pin_3); no longer JG1.6 (Pin_6)
- net GND3: now reaches UT1.9 (GND)
- net GND3: now also UT2.9 (GND)
- net at D12.2 (A), Q12.3 (E): now also JS1.4 (Pin_4); no longer JS1.5 (Pin_5)
- net at D1.2 (A), Q1.3 (E): now also JG1.1 (Pin_1); no longer JG1.8 (Pin_8)
- net at D14.2 (A), Q14.3 (E): now also JS1.6 (Pin_6); no longer JS1.3 (Pin_3)
- net at D5.2 (A), Q5.3 (E): now also JG1.5 (Pin_5); no longer JG1.4 (Pin_4)
- net at D10.2 (A), Q10.3 (E): now also JS1.2 (Pin_2); no longer JS1.7 (Pin_7)
- net at D6.2 (A), Q6.3 (E): now also JG1.6 (Pin_6); no longer JG1.3 (Pin_3)
- net at D13.2 (A), Q13.3 (E): now also JS1.5 (Pin_5); no longer JS1.4 (Pin_4)
- net at D11.2 (A), Q11.3 (E): now also JS1.3 (Pin_3); no longer JS1.6 (Pin_6)
