File: PCB/divergence_meter_logic/divergence_meter_logic.kicad_sch (KiCad schematic)
At the start: 66 parts, among them Q1 BC547, Q10 BC547, Q11 BC547, Q12 BC547, Q13 BC547, Q14 BC547, Q15 BC547, Q16 BC547, Q2 BC547, Q3 BC547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

Commit message: PCB done, exported gerber
Connections:
- net Earth: now reaches H1.1, H2.1, H3.1, H4.1, JP1.2 (C)
Changed lines of the file:
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@@
   (junction (at 25.4 120.65) (diameter 0) (color 0 0 0 0)
   )
-  (junction (at 69.85 167.64) (diameter 0) (color 0 0 0 0)
-  )
   (junction (at 238.76 104.14) (diameter 0) (color 0 0 0 0)
   )
@@
   )
   (junction (at 189.23 134.62) (diameter 0) (color 0 0 0 0)
+  )
+  (junction (at 69.85 186.69) (diameter 0) (color 0 0 0 0)
   )
   (junction (at 189.23 110.49) (diameter 0) (color 0 0 0 0)
@@
     (stroke (width 0) (type default) (color 0 0 0 0))
   )
-  (wire (pts (xy 69.85 160.02) (xy 69.85 167.64))
-    (stroke (width 0) (type default) (color 0 0 0 0))
-  )
   (wire (pts (xy 222.25 140.97) (xy 222.25 134.62))
     (stroke (width 0) (type default) (color 0 0 0 0))
@@
     (stroke (width 0) (type default) (color 0 0 0 0))
   )
+  (wire (pts (xy 69.85 160.02) (xy 69.85 162.56))
+    (stroke (width 0) (type default) (color 0 0 0 0))
+  )
   (wire (pts (xy 246.38 48.26) (xy 246.38 55.88))
     (stroke (width 0) (type default) (color 0 0 0 0))
@@
   )
   (wire (pts (xy 222.25 134.62) (xy 222.25 128.27))
+    (stroke (width 0) (type default) (color 0 0 0 0))
+  )
+  (wire (pts (xy 69.85 186.69) (xy 69.85 189.23))
     (stroke (width 0) (type default) (color 0 0 0 0))
   )
@@
     (pin "1")
   )
+  (symbol (lib_id "power:Earth") (at 69.85 162.56 0) (unit 1)
+    (in_bom yes) (on_board yes) (fields_autoplaced)
+    (property "Reference" "#PWR?" (id 0) (at 69.85 168.91 0)
+      (effects (font (size 1.27 1.27)) hide)
+    )
+    (property "Value" "Earth" (id 1) (at 69.85 166.37 0)
+      (effects (font (size 1.27 1.27)) hide)
+    )
+    (property "Footprint" "" (id 2) (at 69.85 162.56 0)
+      (effects (font (size 1.27 1.27)) hide)
+    )
+    (property "Datasheet" "~" (id 3) (at 69.85 162.56 0)
+      (effects (font (size 1.27 1.27)) hide)
+    )
+    (pin "1")
+  )
   (symbol (lib_id "Transistor_BJT:BC547") (at 210.82 41.91 0) (unit 1)
     (in_bom yes) (on_board yes)
@@
     (pin "1")
   )
+  (symbol (lib_id "power:Earth") (at 69.85 189.23 0) (unit 1)
+    (in_bom yes) (on_board yes) (fields_autoplaced)
+    (property "Reference" "#PWR?" (id 0) (at 69.85 195.58 0)
+      (effects (font (size 1.27 1.27)) hide)
+    )
+    (property "Value" "Earth" (id 1) (at 69.85 193.04 0)
+      (effects (font (size 1.27 1.27)) hide)
+    )
+    (property "Footprint" "" (id 2) (at 69.85 189.23 0)
+      (effects (font (size 1.27 1.27)) hide)
+    )
+    (property "Datasheet" "~" (id 3) (at 69.85 189.23 0)
+      (effects (font (size 1.27 1.27)) hide)
+    )
+    (pin "1")
+  )
   (symbol (lib_id "Device:R") (at 242.57 140.97 90) (mirror x) (unit 1)
     (in_bom yes) (on_board yes)
@@
       (reference "#PWR0124") (unit 1) (value "+1V5") (footprint "")
     )
+    (path "/9a9a81d4-4b02-4e51-b077-4c33c37c3f03"
+      (reference "#PWR?") (unit 1) (value "Earth") (footprint "")
+    )
+    (path "/e28785e6-23a6-4d97-8af1-f33c992f70f8"
+      (reference "#PWR?") (unit 1) (value "Earth") (footprint "")
+    )
     (path "/1cd08355-701e-4fba-886f-d48517dcccf5"
