File: PCB/divergence_meter_logic/divergence_meter_logic.kicad_sch (KiCad schematic)
At the start: 66 parts, among them Q1 BC547, Q10 BC547, Q11 BC547, Q12 BC547, Q13 BC547, Q14 BC547, Q15 BC547, Q16 BC547, Q2 BC547, Q3 BC547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

Commit message: refactoring
Parts:
- removed JL1: Conn_01x10, Connector_PinSocket_2.54mm:PinSocket_1x10_P2.54mm_Vertical, symbol Connector_Generic:Conn_01x10
- removed JP1: SolderJumper_3_Open, Jumper:SolderJumper-3_P1.3mm_Open_RoundedPad1.0x1.5mm_NumberLabels, symbol Jumper:SolderJumper_3_Open
- added C1, C2: 100u, Capacitor_THT:CP_Radial_D5.0mm_P2.00mm, symbol Device:C_Polarized
- added C3: 10u, Capacitor_THT:CP_Radial_D5.0mm_P2.00mm, symbol Device:C_Polarized
- added C4, C5, C6, C7, C8: 100n, Capacitor_THT:C_Disc_D5.0mm_W2.5mm_P5.00mm, symbol Device:C
- added J1: Conn_01x12, Connector_PinSocket_2.54mm:PinSocket_1x12_P2.54mm_Vertical, symbol Connector_Generic:Conn_01x12
- JPWR1: footprint (none) -> Connector_PinHeader_2.54mm:PinHeader_1x08_P2.54mm_Horizontal
- UR1, UR2: footprint SN74HC595N:DIP794W53P254L1930H508Q16N -> Package_DIP:DIP-16_W7.62mm_Socket
- UT1, UT2: footprint ULN2803A:DIP850W46P254L2324H393Q18N -> Package_DIP:DIP-18_W7.62mm_Socket
Connections:
- net Earth is gone; now on net GND: H1.1, H2.1, H3.1, H4.1
- net GND1 is gone; now on net GND: JPWR1.7 (Pin_7)
- net GND3 is gone; now on net GND: JPWR1.2 (Pin_2), UT1.9 (GND), UT2.9 (GND)
- net GNDPWR is gone; now on net GND: JPWR1.8 (Pin_8)
- net +1V5: now also C1.1, J1.11 (Pin_11), J1.12 (Pin_12)
- net +28V: now also C3.1, C7.2, C8.2
- net +5V: now also C2.1, C4.1, C5.1, C6.1
- net GND: now also C1.2, C2.2, C3.2, C4.2, C5.2, C6.2, C7.1, C8.1, J1.10 (Pin_10), J1.9 (Pin_9)
- net at D2.2 (A), Q2.3 (E): now also J1.2 (Pin_2)
- net at D8.2 (A), Q8.3 (E): now also J1.8 (Pin_8)
- net at D4.2 (A), Q4.3 (E): now also J1.4 (Pin_4)
- net at D7.2 (A), Q7.3 (E): now also J1.7 (Pin_7)
- net at D3.2 (A), Q3.3 (E): now also J1.3 (Pin_3)
- net at D1.2 (A), Q1.3 (E): now also J1.1 (Pin_1)
- net at D5.2 (A), Q5.3 (E): now also J1.5 (Pin_5)
- net at D6.2 (A), Q6.3 (E): now also J1.6 (Pin_6)
- no-connect marks 8 -> 19

Commit message: pinout
Connections:
- net at UR1.11 (SRCLK): now also A1.8 (D5); no longer A1.9 (D6)
- net at UR1.12 (RCLK): now also A1.9 (D6); no longer A1.10 (D7)
- net at UR1.14 (SER): now also A1.10 (D7); no longer A1.8 (D5)
Changed lines of the file:
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@@
-    (stroke (width 0) (type default) (color 0 0 0 0))
-  )
-  (wire (pts (xy 78.74 66.04) (xy 135.89 66.04))
     (stroke (width 0) (type default) (color 0 0 0 0))
   )
@@
     (stroke (width 0) (type default) (color 0 0 0 0))
   )
-  (wire (pts (xy 129.54 53.34) (xy 129.54 63.5))
-    (stroke (width 0) (type default) (color 0 0 0 0))
-  )
   (wire (pts (xy 229.87 140.97) (xy 229.87 139.7))
     (stroke (width 0) (type default) (color 0 0 0 0))
@@
     (stroke (width 0) (type default) (color 0 0 0 0))
   )
-  (wire (pts (xy 76.2 60.96) (xy 76.2 74.93))
-    (stroke (width 0) (type default) (color 0 0 0 0))
-  )
   (wire (pts (xy 181.61 110.49) (xy 189.23 110.49))
     (stroke (width 0) (type default) (color 0 0 0 0))
@@
     (stroke (width 0) (type default) (color 0 0 0 0))
   )
+  (wire (pts (xy 73.66 74.93) (xy 73.66 66.04))
+    (stroke (width 0) (type default) (color 0 0 0 0))
+  )
   (wire (pts (xy 115.57 115.57) (xy 135.89 115.57))
     (stroke (width 0) (type default) (color 0 0 0 0))
@@
     (stroke (width 0) (type default) (color 0 0 0 0))
   )
-  (wire (pts (xy 135.89 53.34) (xy 129.54 53.34))
-    (stroke (width 0) (type default) (color 0 0 0 0))
-  )
   (wire (pts (xy 189.23 78.74) (xy 189.23 72.39))
     (stroke (width 0) (type default) (color 0 0 0 0))
   )
+  (wire (pts (xy 76.2 53.34) (xy 76.2 74.93))
+    (stroke (width 0) (type default) (color 0 0 0 0))
+  )
   (wire (pts (xy 246.38 109.22) (xy 246.38 110.49))
     (stroke (width 0) (type default) (color 0 0 0 0))
@@
     (stroke (width 0) (type default) (color 0 0 0 0))
   )
-  (wire (pts (xy 135.89 60.96) (xy 76.2 60.96))
-    (stroke (width 0) (type default) (color 0 0 0 0))
-  )
   (wire (pts (xy 29.21 36.83) (xy 29.21 48.26))
     (stroke (width 0) (type default) (color 0 0 0 0))
@@
     (stroke (width 0) (type default) (color 0 0 0 0))
   )
-  (wire (pts (xy 78.74 74.93) (xy 78.74 66.04))
-    (stroke (width 0) (type default) (color 0 0 0 0))
-  )
   (wire (pts (xy 156.21 50.8) (xy 161.29 50.8))
     (stroke (width 0) (type default) (color 0 0 0 0))
@@
     (stroke (width 0) (type default) (color 0 0 0 0))
   )
+  (wire (pts (xy 78.74 74.93) (xy 78.74 60.96))
+    (stroke (width 0) (type default) (color 0 0 0 0))
+  )
   (wire (pts (xy 156.21 118.11) (xy 161.29 118.11))
     (stroke (width 0) (type default) (color 0 0 0 0))
@@
     (stroke (width 0) (type default) (color 0 0 0 0))
   )
+  (wire (pts (xy 76.2 53.34) (xy 135.89 53.34))
+    (stroke (width 0) (type default) (color 0 0 0 0))
+  )
   (wire (pts (xy 140.97 38.1) (xy 146.05 38.1))
     (stroke (width 0) (type default) (color 0 0 0 0))
@@
     (stroke (width 0) (type default) (color 0 0 0 0))
   )
+  (wire (pts (xy 78.74 60.96) (xy 135.89 60.96))
+    (stroke (width 0) (type default) (color 0 0 0 0))
+  )
   (wire (pts (xy 181.61 96.52) (xy 181.61 107.95))
     (stroke (width 0) (type default) (color 0 0 0 0))
@@
     (stroke (width 0) (type default) (color 0 0 0 0))
   )
+  (wire (pts (xy 73.66 66.04) (xy 135.89 66.04))
+    (stroke (width 0) (type default) (color 0 0 0 0))
+  )
   (wire (pts (xy 246.38 48.26) (xy 246.38 55.88))
     (stroke (width 0) (type default) (color 0 0 0 0))
@@
     (stroke (width 0) (type default) (color 0 0 0 0))
   )
-  (wire (pts (xy 73.66 63.5) (xy 129.54 63.5))
-    (stroke (width 0) (type default) (color 0 0 0 0))
-  )
   (wire (pts (xy 83.82 74.93) (xy 83.82 71.12))
     (stroke (width 0) (type default) (color 0 0 0 0))
   )
-  (wire (pts (xy 73.66 63.5) (xy 73.66 74.93))
-    (stroke (width 0) (type default) (color 0 0 0 0))
-  )
