File: PCB/divergence_meter_logic/divergence_meter_logic.kicad_pcb (KiCad board)
At the start: 2 copper layers, 13 parts

Commit message: remake pcb
Parts:
- JG1, JS1: footprint Connector_PinHeader_2.54mm:PinHeader_1x08_P2.54mm_Vertical -> Connector_PinSocket_2.54mm:PinSocket_1x08_P2.54mm_Vertical
- JRTC1: footprint Connector_PinHeader_2.54mm:PinHeader_1x06_P2.54mm_Vertical -> Connector_PinSocket_2.54mm:PinSocket_1x06_P2.54mm_Vertical
- moved JS1 121.7 mm to (213.4, 76.2)
- moved UT2 121.3 mm to (203.2, 83.8)
- moved UR2 121.2 mm to (201.9, 95.2)
- moved UR1 61.2 mm to (194.3, 119.5)
- moved JR1 61.0 mm to (139.7, 104.1)
- moved JG1 52.2 mm to (167.6, 104.2)
- moved JRTC1 45.5 mm to (85.1, 143.5)
- moved UT1 42.5 mm to (158.8, 104.1)
- moved JPX1 41.6 mm to (62.2, 138.4)
- moved JSW1 41.0 mm to (123.2, 121.9)
- moved JX1 35.8 mm to (106.7, 106.7)
- moved A1 34.6 mm to (139.7, 76.2)
- moved JBT1 22.0 mm to (115.6, 123.2)
Connections:
- A1 pad 10: Net-(A1-Pad10) -> unconnected-(A1-Pad10)
- A1 pad 5: Net-(A1-Pad5) -> unconnected-(A1-Pad5)
- A1 pad 6: Net-(A1-Pad6) -> unconnected-(A1-Pad6)
- A1 pad 7: Net-(A1-Pad7) -> unconnected-(A1-Pad7)
- A1 pad 8: Net-(A1-Pad8) -> unconnected-(A1-Pad8)
- A1 pad 9: Net-(A1-Pad9) -> unconnected-(A1-Pad9)
- JG1 pad 1: Net-(JG1-Pad1) -> Net-(JG1-Pad2)
- JSW1 pad 2: GND -> Net-(JSW1-Pad2)
- JSW1 pad 4: GND -> Net-(JSW1-Pad2)
- JSW1 pad 6: GND -> Net-(JSW1-Pad2)
- UR1 pad 10: +5V -> unconnected-(UR1-Pad10)
- UR1 pad 11: Net-(A1-Pad7) -> unconnected-(UR1-Pad11)
- UR1 pad 12: Net-(A1-Pad6) -> unconnected-(UR1-Pad12)
- UR1 pad 13: GND1 -> unconnected-(UR1-Pad13)
- UR1 pad 14: Net-(A1-Pad5) -> unconnected-(UR1-Pad14)
- UR1 pad 16: +5V -> unconnected-(UR1-Pad16)
- UR1 pad 8: GND1 -> unconnected-(UR1-Pad8)
- UT1 pad 10: Net-(JP3-Pad1) -> unconnected-(UT1-Pad10)
- UT1 pad 11: Net-(JG1-Pad8) -> Net-(UT1-Pad11)
- UT1 pad 12: Net-(JG1-Pad7) -> Net-(UT1-Pad12)
- UT1 pad 13: Net-(JG1-Pad6) -> Net-(UT1-Pad13)
- UT1 pad 14: Net-(JG1-Pad5) -> Net-(UT1-Pad14)
- UT1 pad 15: Net-(JG1-Pad4) -> Net-(UT1-Pad15)
- UT1 pad 16: Net-(JG1-Pad3) -> Net-(UT1-Pad16)
- UT1 pad 17: Net-(JG1-Pad2) -> Net-(UT1-Pad17)
- UT1 pad 18: Net-(JG1-Pad1) -> Net-(UT1-Pad18)

Commit message: blah
Parts:
- added D1: 1N4148, Diode_THT:D_DO-35_SOD27_P2.54mm_Vertical_KathodeUp, F.Cu at (166.4, 133.3)
- added D10: 1N4148, Diode_THT:D_DO-35_SOD27_P2.54mm_Vertical_KathodeUp, F.Cu at (175.2, 101.1)
- added D11: 1N4148, Diode_THT:D_DO-35_SOD27_P2.54mm_Vertical_KathodeUp, F.Cu at (203.2, 94.0)
- added D12: 1N4148, Diode_THT:D_DO-35_SOD27_P2.54mm_Vertical_KathodeUp, F.Cu at (169.2, 101.1)
- added D13: 1N4148, Diode_THT:D_DO-35_SOD27_P2.54mm_Vertical_KathodeUp, F.Cu at (194.3, 90.2)
- added D14: 1N4148, Diode_THT:D_DO-35_SOD27_P2.54mm_Vertical_KathodeUp, F.Cu at (181.7, 95.4)
- added D15: 1N4148, Diode_THT:D_DO-35_SOD27_P2.54mm_Vertical_KathodeUp, F.Cu at (190.5, 101.6)
- added D16: 1N4148, Diode_THT:D_DO-35_SOD27_P2.54mm_Vertical_KathodeUp, F.Cu at (175.7, 95.4)
- added D2: 1N4148, Diode_THT:D_DO-35_SOD27_P2.54mm_Vertical_KathodeUp, F.Cu at (170.2, 141.0)
- added D3: 1N4148, Diode_THT:D_DO-35_SOD27_P2.54mm_Vertical_KathodeUp, F.Cu at (175.3, 130.8)
- added D4: 1N4148, Diode_THT:D_DO-35_SOD27_P2.54mm_Vertical_KathodeUp, F.Cu at (205.7, 143.5)
- added D5: 1N4148, Diode_THT:D_DO-35_SOD27_P2.54mm_Vertical_KathodeUp, F.Cu at (215.9, 124.5)
- added D6: 1N4148, Diode_THT:D_DO-35_SOD27_P2.54mm_Vertical_KathodeUp, F.Cu at (218.4, 113.0)
- added D7: 1N4148, Diode_THT:D_DO-35_SOD27_P2.54mm_Vertical_KathodeUp, F.Cu at (175.3, 135.9)
- added D8: 1N4148, Diode_THT:D_DO-35_SOD27_P2.54mm_Vertical_KathodeUp, F.Cu at (190.5, 127.0)
- added D9: 1N4148, Diode_THT:D_DO-35_SOD27_P2.54mm_Vertical_KathodeUp, F.Cu at (185.4, 105.4)
- added Q1: BC547, Package_TO_SOT_THT:TO-92_Inline, F.Cu at (219.7, 138.4)
- added Q10: BC547, Package_TO_SOT_THT:TO-92_Inline, F.Cu at (218.4, 87.6)
- added Q11: BC547, Package_TO_SOT_THT:TO-92_Inline, F.Cu at (203.2, 87.6)
- added Q12: BC547, Package_TO_SOT_THT:TO-92_Inline, F.Cu at (215.9, 82.5)
- added Q13: BC547, Package_TO_SOT_THT:TO-92_Inline, F.Cu at (205.7, 82.5)
- added Q14: BC547, Package_TO_SOT_THT:TO-92_Inline, F.Cu at (213.4, 87.6)
- added Q15: BC547, Package_TO_SOT_THT:TO-92_Inline, F.Cu at (208.3, 87.6)
- added Q16: BC547, Package_TO_SOT_THT:TO-92_Inline, F.Cu at (210.8, 82.5)
- added Q2: BC547, Package_TO_SOT_THT:TO-92_Inline, F.Cu at (198.1, 142.2)
- added Q3: BC547, Package_TO_SOT_THT:TO-92_Inline, F.Cu at (214.6, 130.8)
- added Q4: BC547, Package_TO_SOT_THT:TO-92_Inline, F.Cu at (212.1, 138.4)
- added Q5: BC547, Package_TO_SOT_THT:TO-92_Inline, F.Cu at (204.5, 135.9)
- added Q6: BC547, Package_TO_SOT_THT:TO-92_Inline, F.Cu at (190.5, 135.9)
- added Q7: BC547, Package_TO_SOT_THT:TO-92_Inline, F.Cu at (198.1, 133.3)
- added Q8: BC547, Package_TO_SOT_THT:TO-92_Inline, F.Cu at (205.7, 127.0)
- added Q9: BC547, Package_TO_SOT_THT:TO-92_Inline, F.Cu at (200.7, 82.5)
- added R1: 100k, Resistor_THT:R_Axial_DIN0204_L3.6mm_D1.6mm_P2.54mm_Vertical, F.Cu at (176.5, 143.5)
- added R10: 100k, Resistor_THT:R_Axial_DIN0204_L3.6mm_D1.6mm_P2.54mm_Vertical, F.Cu at (186.7, 76.2)
- added R11: 100k, Resistor_THT:R_Axial_DIN0204_L3.6mm_D1.6mm_P2.54mm_Vertical, F.Cu at (210.8, 101.6)
- added R12: 100k, Resistor_THT:R_Axial_DIN0204_L3.6mm_D1.6mm_P2.54mm_Vertical, F.Cu at (210.8, 92.7)
- added R13: 100k, Resistor_THT:R_Axial_DIN0204_L3.6mm_D1.6mm_P2.54mm_Vertical, F.Cu at (181.2, 98.8)
- added R14: 100k, Resistor_THT:R_Axial_DIN0204_L3.6mm_D1.6mm_P2.54mm_Vertical, F.Cu at (217.2, 100.3)
- added R15: 100k, Resistor_THT:R_Axial_DIN0204_L3.6mm_D1.6mm_P2.54mm_Vertical, F.Cu at (199.4, 101.6)
- added R16: 100k, Resistor_THT:R_Axial_DIN0204_L3.6mm_D1.6mm_P2.54mm_Vertical, F.Cu at (187.7, 92.9)
- added R2: 100k, Resistor_THT:R_Axial_DIN0204_L3.6mm_D1.6mm_P2.54mm_Vertical, F.Cu at (186.7, 141.0)
- added R3: 100k, Resistor_THT:R_Axial_DIN0204_L3.6mm_D1.6mm_P2.54mm_Vertical, F.Cu at (240.0, 129.5)
- added R4: 100k, Resistor_THT:R_Axial_DIN0204_L3.6mm_D1.6mm_P2.54mm_Vertical, F.Cu at (166.4, 144.8)
- added R5: 100k, Resistor_THT:R_Axial_DIN0204_L3.6mm_D1.6mm_P2.54mm_Vertical, F.Cu at (182.9, 134.6)
- added R6: 100k, Resistor_THT:R_Axial_DIN0204_L3.6mm_D1.6mm_P2.54mm_Vertical, F.Cu at (182.9, 127.0)
- added R7: 100k, Resistor_THT:R_Axial_DIN0204_L3.6mm_D1.6mm_P2.54mm_Vertical, F.Cu at (226.1, 114.3)
- added R8: 100k, Resistor_THT:R_Axial_DIN0204_L3.6mm_D1.6mm_P2.54mm_Vertical, F.Cu at (199.4, 123.2)
- added R9: 100k, Resistor_THT:R_Axial_DIN0204_L3.6mm_D1.6mm_P2.54mm_Vertical, F.Cu at (198.1, 106.7)
- UT1, UT2: moved to F.Cu
- moved JPX1 98.9 mm to (118.5, 57.1)
- moved JRTC1 91.7 mm to (101.6, 53.3)
- moved UT2 70.0 mm to (133.3, 87.8), turned to 0 degrees
- moved JG1 62.7 mm to (227.3, 123.2), turned to 0 degrees
- moved UR1 61.7 mm to (133.2, 110.8), turned to 0 degrees
- moved UR2 59.8 mm to (144.2, 110.8), turned to 0 degrees
- moved JSW1 59.5 mm to (143.5, 66.0)
- moved JX1 49.5 mm to (82.5, 63.5)
- moved JBT1 43.4 mm to (152.3, 100.2)
- moved JR1 35.7 mm to (110.8, 125.0)
- moved A1 29.5 mm to (110.5, 80.0), turned to 0 degrees
- moved UT1 21.7 mm to (144.4, 87.8), turned to 0 degrees
- moved JS1 12.7 mm to (200.7, 76.2), turned to 90 degrees
Connections:
- A1 pad 13: Net-(A1-Pad13) -> unconnected-(A1-Pad13)
- A1 pad 14: Net-(A1-Pad14) -> unconnected-(A1-Pad14)
- A1 pad 15: Net-(A1-Pad15) -> unconnected-(A1-Pad15)
- JG1 pad 1: Net-(JG1-Pad2) -> Net-(D1-Pad2)
- JG1 pad 2: Net-(JG1-Pad2) -> Net-(D3-Pad2)
- JS1 pad 1: Net-(JS1-Pad1) -> Net-(D9-Pad2)
- JS1 pad 2: Net-(JS1-Pad2) -> Net-(D11-Pad2)
- JS1 pad 3: Net-(JS1-Pad3) -> Net-(D13-Pad2)
- JS1 pad 4: Net-(JS1-Pad4) -> Net-(D15-Pad2)
- JS1 pad 5: Net-(JS1-Pad5) -> Net-(D16-Pad2)
- JS1 pad 6: Net-(JS1-Pad6) -> Net-(D14-Pad2)
- JS1 pad 7: Net-(JS1-Pad7) -> Net-(D12-Pad2)
- JS1 pad 8: Net-(JS1-Pad8) -> Net-(D10-Pad2)
- UR1 pad 10: unconnected-(UR1-Pad10) -> +5V
- UR1 pad 13: unconnected-(UR1-Pad13) -> GND1
- UR1 pad 16: unconnected-(UR1-Pad16) -> +5V
- UR1 pad 8: unconnected-(UR1-Pad8) -> GND1
- UR2 pad 11: Net-(A1-Pad10) -> unconnected-(UR2-Pad11)
- UR2 pad 12: Net-(A1-Pad9) -> unconnected-(UR2-Pad12)
- UR2 pad 14: Net-(A1-Pad8) -> unconnected-(UR2-Pad14)
- UT1 pad 10: unconnected-(UT1-Pad10) -> +28V
- UT2 pad 10: Net-(JP3-Pad1) -> +28V
- UT2 pad 11: Net-(JS1-Pad8) -> Net-(D10-Pad1)
- UT2 pad 12: Net-(JS1-Pad7) -> Net-(D12-Pad1)
- UT2 pad 13: Net-(JS1-Pad6) -> Net-(D14-Pad1)
- UT2 pad 14: Net-(JS1-Pad5) -> Net-(D16-Pad1)
- UT2 pad 15: Net-(JS1-Pad4) -> Net-(D15-Pad1)
- UT2 pad 16: Net-(JS1-Pad3) -> Net-(D13-Pad1)
- UT2 pad 17: Net-(JS1-Pad2) -> Net-(D11-Pad1)
- UT2 pad 18: Net-(JS1-Pad1) -> Net-(D9-Pad1)

Commit message: wuzah
Parts:
- UR2: moved to B.Cu
- moved UT1 53.4 mm to (143.3, 141.2)
- moved UT2 53.1 mm to (186.4, 88.4)
- moved D12 49.0 mm to (213.4, 79.8)
- moved D10 41.4 mm to (215.9, 93.5)
- moved R10 40.0 mm to (218.4, 100.6), turned to 180 degrees
- moved UR2 36.5 mm to (173.7, 89.4), turned to 180 degrees
- moved D16 35.2 mm to (207.3, 79.8)
- moved A1 30.5 mm to (140.7, 76.2), turned to -90 degrees
- moved UR1 29.0 mm to (130.0, 139.7), turned to 180 degrees
- moved D14 27.9 mm to (209.6, 93.5)
- moved D9 27.4 mm to (195.1, 79.8)
- moved R13 25.5 mm to (203.7, 86.9), turned to 180 degrees
- moved R16 22.9 mm to (209.8, 86.9), turned to 180 degrees
- moved R9 19.8 mm to (197.6, 86.9), turned to 180 degrees
- moved D15 14.7 mm to (202.7, 93.5)
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Connections:
- UT1 pad 1: Net-(UR1-Pad15) -> Net-(UR1-Pad7)
- UT1 pad 2: Net-(UR1-Pad1) -> Net-(UR1-Pad6)
- UT1 pad 3: Net-(UR1-Pad2) -> Net-(UR1-Pad5)
- UT1 pad 4: Net-(UR1-Pad3) -> Net-(UR1-Pad4)
- UT1 pad 5: Net-(UR1-Pad4) -> Net-(UR1-Pad3)
- UT1 pad 6: Net-(UR1-Pad5) -> Net-(UR1-Pad2)
- UT1 pad 7: Net-(UR1-Pad6) -> Net-(UR1-Pad1)
- UT1 pad 8: Net-(UR1-Pad7) -> Net-(UR1-Pad15)
- UT2 pad 11: Net-(D10-Pad1) -> Net-(D9-Pad1)
- UT2 pad 12: Net-(D12-Pad1) -> Net-(D11-Pad1)
- UT2 pad 13: Net-(D14-Pad1) -> Net-(D13-Pad1)
- UT2 pad 14: Net-(D16-Pad1) -> Net-(D15-Pad1)
- UT2 pad 15: Net-(D15-Pad1) -> Net-(D16-Pad1)
- UT2 pad 16: Net-(D13-Pad1) -> Net-(D14-Pad1)
- UT2 pad 17: Net-(D11-Pad1) -> Net-(D12-Pad1)
- UT2 pad 18: Net-(D9-Pad1) -> Net-(D10-Pad1)
Routing:
- net +28V: track 0.00 -> 34.7 mm
- net Net-(D11-Pad2): track 0.00 -> 13.8 mm
- net Net-(D15-Pad2): track 0.00 -> 12.7 mm
- net Net-(D14-Pad2): track 0.00 -> 12.3 mm
- net Net-(D9-Pad2): track 0.00 -> 8.88 mm
- net Net-(D13-Pad2): track 0.00 -> 8.46 mm
- net Net-(D16-Pad1): track 0.00 -> 8.16 mm
- net Net-(D13-Pad1): track 0.00 -> 8.16 mm
- net Net-(D9-Pad1): track 0.00 -> 8.16 mm
- net Net-(D12-Pad1): track 0.00 -> 8.16 mm
- net Net-(D12-Pad2): track 0.00 -> 7.62 mm
- net Net-(D16-Pad2): track 0.00 -> 3.98 mm

Commit message: pcb rework
Parts:
- removed JBT1: Conn_01x06, Connector_PinHeader_2.54mm:PinHeader_1x06_P2.54mm_Vertical
- removed JPX1: Conn_02x04_Odd_Even, Connector_PinHeader_2.54mm:PinHeader_2x04_P2.54mm_Vertical
- removed JR1: Conn_01x02, Connector_PinHeader_2.54mm:PinHeader_1x02_P2.54mm_Vertical
- removed JSW1: Conn_02x03_Odd_Even, Connector_PinHeader_2.54mm:PinHeader_2x03_P2.54mm_Vertical
- removed JX1: Conn_01x07, Connector_PinHeader_2.54mm:PinHeader_1x07_P2.54mm_Vertical
- added H1: MountingHole_Pad, MountingHole:MountingHole_3.5mm_Pad_Via, F.Cu at (176.8, 69.6)
- added H2: MountingHole_Pad, MountingHole:MountingHole_3.5mm_Pad_Via, F.Cu at (185.3, 68.4)
- added H3: MountingHole_Pad, MountingHole:MountingHole_3.5mm_Pad_Via, F.Cu at (181.4, 59.9)
- added H4: MountingHole_Pad, MountingHole:MountingHole_3.5mm_Pad_Via, F.Cu at (190.0, 59.9)
- added JGND1: Conn_01x03, Connector_PinHeader_2.54mm:PinHeader_1x03_P2.54mm_Vertical, F.Cu at (174.8, 57.9)
- UR2: moved to F.Cu
- moved UR2 2.74 mm to (172.7, 86.9)
- moved JS1 2.54 mm to (198.1, 76.2)
- moved UR1 0.51 mm to (130.6, 139.7)
- renumbered D12 to D10, D14 to D11, D16 to D12, D15 to D13, D13 to D14, D11 to D15, D9 to D16, D3 to D2, D5 to D3, D7 to D4, D8 to D5, D4 to D7, D2 to D8, D10 to D9, Q12 to Q10, Q14 to Q11, Q16 to Q12, Q15 to Q13, Q13 to Q14, Q11 to Q15, Q9 to Q16, Q3 to Q2, Q5 to Q3, Q7 to Q4, Q8 to Q5, Q4 to Q7, Q2 to Q8, Q10 to Q9, R12 to R10, R14 to R11, R16 to R12, R15 to R13, R13 to R14, R11 to R15, R9 to R16, R3 to R2, R5 to R3, R7 to R4, R8 to R5, R4 to R7, R2 to R8, R10 to R9
Connections:
- A1 pad 10: unconnected-(A1-Pad10) -> Net-(UR1-Pad11)
- A1 pad 11: Net-(A1-Pad11) -> unconnected-(A1-Pad11)
- A1 pad 12: Net-(A1-Pad12) -> unconnected-(A1-Pad12)
- A1 pad 16: Net-(A1-Pad16) -> unconnected-(A1-Pad16)
- A1 pad 21: Net-(A1-Pad21) -> unconnected-(A1-Pad21)
- A1 pad 22: Net-(A1-Pad22) -> unconnected-(A1-Pad22)
- A1 pad 23: Net-(A1-Pad23) -> unconnected-(A1-Pad23)
- A1 pad 24: Net-(A1-Pad24) -> unconnected-(A1-Pad24)
- A1 pad 25: Net-(A1-Pad25) -> unconnected-(A1-Pad25)
- A1 pad 26: Net-(A1-Pad26) -> unconnected-(A1-Pad26)
- A1 pad 29: GND1 -> GND
- A1 pad 4: GND1 -> unconnected-(A1-Pad4)
- A1 pad 5: unconnected-(A1-Pad5) -> Net-(UR2-Pad14)
- A1 pad 6: unconnected-(A1-Pad6) -> Net-(UR2-Pad12)
- A1 pad 7: unconnected-(A1-Pad7) -> Net-(UR2-Pad11)
- A1 pad 8: unconnected-(A1-Pad8) -> Net-(UR1-Pad14)
- A1 pad 9: unconnected-(A1-Pad9) -> Net-(UR1-Pad12)
- D10 pad 2: Net-(D12-Pad2) -> Net-(D10-Pad2)
- D11 pad 2: Net-(D14-Pad2) -> Net-(D11-Pad2)
- D12 pad 2: Net-(D16-Pad2) -> Net-(D12-Pad2)
- D13 pad 2: Net-(D15-Pad2) -> Net-(D13-Pad2)
- D14 pad 2: Net-(D13-Pad2) -> Net-(D14-Pad2)
- D15 pad 2: Net-(D11-Pad2) -> Net-(D15-Pad2)
- D16 pad 2: Net-(D9-Pad2) -> Net-(D16-Pad2)
- D9 pad 2: Net-(D10-Pad2) -> Net-(D9-Pad2)
- JRTC1 pad 1: GND1 -> GND
- JS1 pad 2: Net-(D11-Pad2) -> Net-(D10-Pad2)
- JS1 pad 3: Net-(D13-Pad2) -> Net-(D11-Pad2)
- JS1 pad 4: Net-(D15-Pad2) -> Net-(D12-Pad2)
- JS1 pad 5: Net-(D16-Pad2) -> Net-(D13-Pad2)
- JS1 pad 7: Net-(D12-Pad2) -> Net-(D15-Pad2)
- JS1 pad 8: Net-(D10-Pad2) -> Net-(D16-Pad2)
- Q10 pad 3: Net-(D12-Pad2) -> Net-(D10-Pad2)
- Q11 pad 3: Net-(D14-Pad2) -> Net-(D11-Pad2)
- Q12 pad 3: Net-(D16-Pad2) -> Net-(D12-Pad2)
- Q13 pad 3: Net-(D15-Pad2) -> Net-(D13-Pad2)
- Q14 pad 3: Net-(D13-Pad2) -> Net-(D14-Pad2)
- Q15 pad 3: Net-(D11-Pad2) -> Net-(D15-Pad2)
- Q16 pad 3: Net-(D9-Pad2) -> Net-(D16-Pad2)
- Q9 pad 3: Net-(D10-Pad2) -> Net-(D9-Pad2)
- UR1 pad 11: unconnected-(UR1-Pad11) -> Net-(UR1-Pad11)
- UR1 pad 12: unconnected-(UR1-Pad12) -> Net-(UR1-Pad12)
- UR1 pad 13: GND1 -> GND
- UR1 pad 14: unconnected-(UR1-Pad14) -> Net-(UR1-Pad14)
- UR1 pad 8: GND1 -> GND
- UR2 pad 1: Net-(UR2-Pad1) -> Net-(UT2-Pad7)
- UR2 pad 11: unconnected-(UR2-Pad11) -> Net-(UR2-Pad11)
- UR2 pad 12: unconnected-(UR2-Pad12) -> Net-(UR2-Pad12)
- UR2 pad 13: GND1 -> GND
- UR2 pad 14: unconnected-(UR2-Pad14) -> Net-(UR2-Pad14)
- UR2 pad 15: Net-(UR2-Pad15) -> Net-(UT2-Pad8)
- UR2 pad 2: Net-(UR2-Pad2) -> Net-(UT2-Pad6)
- UR2 pad 3: Net-(UR2-Pad3) -> Net-(UT2-Pad5)
- UR2 pad 4: Net-(UR2-Pad4) -> Net-(UT2-Pad4)
- UR2 pad 5: Net-(UR2-Pad5) -> Net-(UT2-Pad3)
- UR2 pad 6: Net-(UR2-Pad6) -> Net-(UT2-Pad2)
- UR2 pad 7: Net-(UR2-Pad7) -> Net-(UT2-Pad1)
- UR2 pad 8: GND1 -> GND
- UT1 pad 9: GND -> unconnected-(UT1-Pad9)
- UT2 pad 1: Net-(UR2-Pad15) -> Net-(UT2-Pad1)
- UT2 pad 2: Net-(UR2-Pad1) -> Net-(UT2-Pad2)
- UT2 pad 3: Net-(UR2-Pad2) -> Net-(UT2-Pad3)
- UT2 pad 4: Net-(UR2-Pad3) -> Net-(UT2-Pad4)
- UT2 pad 5: Net-(UR2-Pad4) -> Net-(UT2-Pad5)
- UT2 pad 6: Net-(UR2-Pad5) -> Net-(UT2-Pad6)
- UT2 pad 7: Net-(UR2-Pad6) -> Net-(UT2-Pad7)
- UT2 pad 8: Net-(UR2-Pad7) -> Net-(UT2-Pad8)
- UT2 pad 9: GND -> unconnected-(UT2-Pad9)
Routing:
- net Net-(D9-Pad2): track 8.88 -> 0.00 mm
- net Net-(D12-Pad2): track 7.62 -> 0.00 mm
- net Net-(D10-Pad2): track 0.00 -> 7.62 mm
- net Net-(D16-Pad2): track 3.98 -> 8.88 mm
- net Net-(D13-Pad2): track 8.46 -> 12.7 mm

Commit message: pcb finishing
Parts:
- removed JGND1: Conn_01x03, Connector_PinHeader_2.54mm:PinHeader_1x03_P2.54mm_Vertical
- added JP1: SolderJumper_3_Open, Jumper:SolderJumper-3_P1.3mm_Open_RoundedPad1.0x1.5mm_NumberLabels, F.Cu at (103.6, 117.3)
- JRTC1: footprint Connector_PinSocket_2.54mm:PinSocket_1x06_P2.54mm_Vertical -> Connector_PinSocket_2.54mm:PinSocket_1x06_P2.54mm_Horizontal
- moved H4 112.9 mm to (92.5, 116.8)
- moved R2 101.0 mm to (147.3, 89.4)
- moved H1 86.1 mm to (90.9, 63.5)
- moved JG1 84.9 mm to (145.8, 112.8), turned to 90 degrees
- moved Q1 82.4 mm to (145.0, 103.6), turned to 180 degrees
- moved R4 76.5 mm to (153.7, 89.4)
- moved Q2 75.5 mm to (149.6, 92.5), turned to 180 degrees
- moved UR1 74.3 mm to (178.3, 82.8), turned to 0 degrees
- moved JRTC1 67.7 mm to (133.1, 113.3), turned to -90 degrees
- moved D3 66.2 mm to (151.9, 107.7), turned to 180 degrees
- moved H3 64.7 mm to (217.9, 113.3)
- moved UT1 63.1 mm to (157.5, 79.8), turned to -90 degrees
- moved Q3 61.7 mm to (151.9, 103.6), turned to 180 degrees
- moved Q4 58.6 mm to (156.2, 92.5), turned to 180 degrees
- moved Q7 58.5 mm to (165.1, 103.6), turned to 180 degrees
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Connections:
- A1 pad 4: unconnected-(A1-Pad4) -> GND
- UT1 pad 11: Net-(D8-Pad1) -> Net-(D1-Pad1)
- UT1 pad 12: Net-(D7-Pad1) -> Net-(D2-Pad1)
- UT1 pad 13: Net-(D6-Pad1) -> Net-(D3-Pad1)
- UT1 pad 14: Net-(D5-Pad1) -> Net-(D4-Pad1)
- UT1 pad 15: Net-(D4-Pad1) -> Net-(D5-Pad1)
- UT1 pad 16: Net-(D3-Pad1) -> Net-(D6-Pad1)
- UT1 pad 17: Net-(D2-Pad1) -> Net-(D7-Pad1)
- UT1 pad 18: Net-(D1-Pad1) -> Net-(D8-Pad1)
- UT1 pad 9: unconnected-(UT1-Pad9) -> GND3
- UT2 pad 11: Net-(D16-Pad1) -> Net-(D9-Pad1)
- UT2 pad 12: Net-(D15-Pad1) -> Net-(D10-Pad1)
- UT2 pad 13: Net-(D14-Pad1) -> Net-(D11-Pad1)
- UT2 pad 14: Net-(D13-Pad1) -> Net-(D12-Pad1)
- UT2 pad 15: Net-(D12-Pad1) -> Net-(D13-Pad1)
- UT2 pad 16: Net-(D11-Pad1) -> Net-(D14-Pad1)
- UT2 pad 17: Net-(D10-Pad1) -> Net-(D15-Pad1)
- UT2 pad 18: Net-(D9-Pad1) -> Net-(D16-Pad1)
- UT2 pad 9: unconnected-(UT2-Pad9) -> GND3
Routing:
- net +28V: track 34.7 -> 0.00 mm
- net Net-(D11-Pad2): track 13.8 -> 0.00 mm
- net Net-(D13-Pad2): track 12.7 -> 0.00 mm
- net Net-(D14-Pad2): track 12.4 -> 0.00 mm
- net Net-(D15-Pad2): track 12.3 -> 0.00 mm
- net Net-(D16-Pad2): track 8.88 -> 0.00 mm
- net Net-(D14-Pad1): track 8.16 -> 0.00 mm
- net Net-(D12-Pad1): track 8.16 -> 0.00 mm
- net Net-(D16-Pad1): track 8.16 -> 0.00 mm
- net Net-(D10-Pad1): track 8.16 -> 0.00 mm
- net Net-(D10-Pad2): track 7.62 -> 0.00 mm
