File: PCB/divergence_meter_logic/divergence_meter_logic.kicad_pcb (KiCad board)
At the start: 2 copper layers, 137.7 x 56.4 mm, 66 parts, among them Q1 BC547, Q10 BC547, Q11 BC547, Q12 BC547, Q13 BC547, Q14 BC547, Q15 BC547, Q16 BC547, Q2 BC547, Q3 BC547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

Commit message: refactoring
Parts:
- removed JL1: Conn_01x10, Connector_PinSocket_2.54mm:PinSocket_1x10_P2.54mm_Vertical
- removed JP1: SolderJumper_3_Open, Jumper:SolderJumper-3_P1.3mm_Open_RoundedPad1.0x1.5mm_NumberLabels
- added C1: 100u, Capacitor_THT:CP_Radial_D5.0mm_P2.00mm, F.Cu at (97.5, 71.1)
- added C2: 100u, Capacitor_THT:CP_Radial_D5.0mm_P2.00mm, F.Cu at (90.0, 71.1)
- added C3: 10u, Capacitor_THT:CP_Radial_D5.0mm_P2.00mm, F.Cu at (146.8, 61.0)
- added C4: 100n, Capacitor_THT:C_Disc_D5.0mm_W2.5mm_P5.00mm, F.Cu at (121.8, 105.7)
- added C5: 100n, Capacitor_THT:C_Disc_D5.0mm_W2.5mm_P5.00mm, F.Cu at (190.6, 84.3)
- added C6: 100n, Capacitor_THT:C_Disc_D5.0mm_W2.5mm_P5.00mm, F.Cu at (190.6, 63.0)
- added C7: 100n, Capacitor_THT:C_Disc_D5.0mm_W2.5mm_P5.00mm, F.Cu at (151.1, 66.8)
- added C8: 100n, Capacitor_THT:C_Disc_D5.0mm_W2.5mm_P5.00mm, F.Cu at (216.5, 105.3)
- added J1: Conn_01x12, Connector_PinSocket_2.54mm:PinSocket_1x12_P2.54mm_Vertical, F.Cu at (152.4, 109.2)
- JPWR1: value Conn_01x07 -> Conn_01x08; footprint Connector_PinHeader_2.54mm:PinHeader_1x07_P2.54mm_Horizontal -> Connector_PinHeader_2.54mm:PinHeader_1x08_P2.54mm_Horizontal
- UR1, UR2: footprint SN74HC595N:DIP794W53P254L1930H508Q16N -> Package_DIP:DIP-16_W7.62mm_Socket
- UT1, UT2: footprint ULN2803A:DIP850W46P254L2324H393Q18N -> Package_DIP:DIP-18_W7.62mm_Socket
- moved UT1 16.3 mm to (174.7, 67.1)
- moved UT2 10.5 mm to (193.0, 108.5)
- moved UR2 9.16 mm to (179.8, 84.8), turned to 0 degrees
- moved UR1 7.74 mm to (179.8, 63.5)
- moved D11 5.35 mm to (212.6, 86.5)
- moved D12 5.35 mm to (210.6, 72.8)
- moved D13 5.35 mm to (206.0, 86.5)
- moved D14 5.35 mm to (204.0, 72.8)
- moved D15 5.35 mm to (199.5, 86.5)
- moved D16 5.35 mm to (197.4, 72.8)
- moved D9 5.35 mm to (219.2, 86.5)
- moved Q11 5.35 mm to (212.6, 90.6)
- moved Q12 5.35 mm to (210.6, 76.8)
- moved Q13 5.35 mm to (206.0, 90.6)
- moved Q14 5.35 mm to (204.0, 76.8)
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Connections:
- H1 pad 1: Earth -> GND
- H2 pad 1: Earth -> GND
- H3 pad 1: Earth -> GND
- H4 pad 1: Earth -> GND
- JPWR1 pad 2: GND3 -> GND
- JPWR1 pad 6: GND1 -> +1V5
- JPWR1 pad 7: GNDPWR -> GND
- UT1 pad 9: GND3 -> GND
- UT2 pad 9: GND3 -> GND
Routing:
- net GND3: track 154.7 -> 0.00 mm
- net GND: track 249.9 -> 134.0 mm, vias 0 -> 36
- net GND1: track 100.4 -> 0.00 mm, vias 1 -> 0
- net +28V: track 266.8 -> 342.6 mm, vias 0 -> 2
- net +5V: track 166.0 -> 222.1 mm, vias 2 -> 5
- net Net-(A1-Pad5): track 52.8 -> 85.9 mm, vias 0 -> 2
- net Net-(A1-Pad6): track 54.5 -> 83.3 mm, vias 0 -> 2
- net Net-(A1-Pad7): track 58.8 -> 81.6 mm, vias 0 -> 1
- net Net-(UR2-Pad1): track 24.6 -> 46.4 mm
- net +1V5: track 99.0 -> 118.6 mm, vias 1 -> 2
- net Net-(A1-Pad9): track 56.6 -> 75.1 mm, vias 0 -> 4
- net Net-(A1-Pad10): track 54.5 -> 71.8 mm, vias 0 -> 4
- net Net-(UR2-Pad2): track 26.6 -> 41.6 mm
- net Net-(UR2-Pad7): track 32.4 -> 18.1 mm
- net GNDPWR: track 10.1 -> 0.00 mm
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- added copper zone on B.Cu, net GND
- added copper zone on F.Cu, net GND
- removed copper zone on B.Cu, net Earth
- removed copper zone on F.Cu, net Earth

Commit message: pinout
Connections:
- A1 pad 10: Net-(A1-Pad10) -> Net-(UR1-Pad14)
- A1 pad 8: Net-(A1-Pad8) -> Net-(UR1-Pad11)
- A1 pad 9: Net-(A1-Pad9) -> Net-(UR1-Pad12)
- UR1 pad 11: Net-(A1-Pad9) -> Net-(UR1-Pad11)
- UR1 pad 12: Net-(A1-Pad10) -> Net-(UR1-Pad12)
- UR1 pad 14: Net-(A1-Pad8) -> Net-(UR1-Pad14)
Routing:
- net Net-(A1-Pad9): track 75.1 -> 0.00 mm, vias 4 -> 0
- net Net-(A1-Pad10): track 71.8 -> 0.00 mm, vias 4 -> 0
- net Net-(A1-Pad8): track 69.1 -> 0.00 mm, vias 4 -> 0
- net Net-(UR1-Pad11): track 0.00 -> 53.4 mm
- net Net-(UR1-Pad12): track 0.00 -> 50.9 mm
- net Net-(UR1-Pad14): track 0.00 -> 50.5 mm
- net GND: track 134.0 -> 159.5 mm, vias 36 -> 39
- net +5V: track 222.1 -> 222.5 mm, vias 5 -> 3
