File: PCB/review/PCBv2(1)/PCB/divergence_meter_logic/divergence_meter_logic.kicad_pcb (KiCad board)
At the start: 2 copper layers, 137.7 x 56.4 mm, 73 parts, among them J1 Conn_01x12, Q1 BC547, Q10 BC547, Q11 BC547, Q12 BC547, Q13 BC547, Q14 BC547, Q15 BC547, Q16 BC547, Q2 BC547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

Commit message: reviewed, schemes ok
Routing:
- net GND: track 134.0 -> 94.6 mm, vias 36 -> 35
- net Net-(A1-Pad7): track 81.6 -> 80.5 mm
- net Net-(A1-Pad5): track 85.9 -> 84.8 mm
- net Net-(A1-Pad6): track 83.3 -> 82.2 mm
