File: PCB/review/v2/PCB/divergence_meter_top (another copy)/divergence_meter_top.kicad_pcb (KiCad board)
At the start: 2 copper layers, 137.7 x 56.4 mm, 14 parts

Commit message: reviewed, schemes ok
Connections:
- net Net-(JT2-Pad1) renamed B
- net Net-(JT2-Pad2) renamed A
- net Net-(JT2-Pad3) renamed G
- net Net-(JT2-Pad4) renamed F
- net Net-(JT2-Pad5) renamed E
- net Net-(JT2-Pad6) renamed D
- net Net-(JT2-Pad7) renamed C
- net Net-(JT2-Pad8) renamed DP
- net Net-(itr1-Pad9) renamed Gr1
- net Net-(itr2-Pad9) renamed Gr2
- net Net-(itr3-Pad9) renamed Gr3
- net Net-(itr4-Pad9) renamed Gr4
- net Net-(itr5-Pad9) renamed Gr5
- net Net-(itr6-Pad9) renamed Gr6
- net Net-(itr7-Pad9) renamed Gr7
- net Net-(itr8-Pad9) renamed Gr8
Routing:
- net +1V5: track 142.0 -> 143.6 mm, vias 1 -> 2
- net GND: vias 21 -> 19
